File: pool-piano-synth.kicad_pcb (KiCad board)
At the start: 2 copper layers, 88.1 x 72.9 mm, 21 parts, among them J1 Screw_Terminal_01x02, J2 Screw_Terminal_01x02, U1 6N138, U2 ESP32-DevKitC, U3 Teensy4.1

Commit message: v0: ready to print
- add traces, zones, better footprints
Parts:
- removed REF** (x4): PinHeader_1x20_P2.54mm_Vertical, Connector_PinHeader_2.54mm:PinHeader_1x20_P2.54mm_Vertical
- removed REF**: PinHeader_1x02_P2.54mm_Vertical, Connector_PinHeader_2.54mm:PinHeader_1x02_P2.54mm_Vertical
- removed REF**: PinSocket_1x01_P2.54mm_Vertical, Connector_PinSocket_2.54mm:PinSocket_1x01_P2.54mm_Vertical
- added J3: Conn_01x01_Male, Connector_PinHeader_2.54mm:PinHeader_1x01_P2.54mm_Vertical, F.Cu at (168.7, 75.9)
- added J4: Conn_01x20_Male, Connector_PinHeader_2.54mm:PinHeader_1x20_P2.54mm_Vertical, F.Cu at (220.2, 85.3)
- added J5: Conn_01x20_Male, Connector_PinHeader_2.54mm:PinHeader_1x20_P2.54mm_Vertical, F.Cu at (217.7, 85.3)
- added J6: Conn_01x20_Male, Connector_PinHeader_2.54mm:PinHeader_1x20_P2.54mm_Vertical, F.Cu at (215.1, 85.3)
- added J7: Conn_01x20_Male, Connector_PinHeader_2.54mm:PinHeader_1x20_P2.54mm_Vertical, F.Cu at (225.3, 85.3)
- added J8: Conn_01x02_Male, Connector_PinHeader_2.54mm:PinHeader_1x02_P2.54mm_Vertical, F.Cu at (168.7, 131.8)
- C1: footprint Capacitor_THT:CP_Radial_D8.0mm_P5.00mm -> Capacitor_THT:CP_Radial_D10.0mm_P5.00mm
Connections:
- U2 pad 1: unconnected-(U2-Pad1) -> Net-(U2-Pad1)
- U2 pad 10: unconnected-(U2-Pad10) -> Net-(U2-Pad10)
- U2 pad 11: unconnected-(U2-Pad11) -> Net-(U2-Pad11)
- U2 pad 12: unconnected-(U2-Pad12) -> Net-(U2-Pad12)
- U2 pad 13: unconnected-(U2-Pad13) -> Net-(U2-Pad13)
- U2 pad 14: unconnected-(U2-Pad14) -> Net-(U2-Pad14)
- U2 pad 15: unconnected-(U2-Pad15) -> Net-(U2-Pad15)
- U2 pad 16: unconnected-(U2-Pad16) -> Net-(U2-Pad16)
- U2 pad 17: unconnected-(U2-Pad17) -> Net-(U2-Pad17)
- U2 pad 18: unconnected-(U2-Pad18) -> Net-(U2-Pad18)
- U2 pad 2: unconnected-(U2-Pad2) -> Net-(U2-Pad2)
- U2 pad 3: unconnected-(U2-Pad3) -> Net-(U2-Pad3)
- U2 pad 4: unconnected-(U2-Pad4) -> Net-(U2-Pad4)
- U2 pad 5: unconnected-(U2-Pad5) -> Net-(U2-Pad5)
- U2 pad 6: unconnected-(U2-Pad6) -> Net-(U2-Pad6)
- U2 pad 7: unconnected-(U2-Pad7) -> Net-(U2-Pad7)
- U2 pad 8: unconnected-(U2-Pad8) -> Net-(U2-Pad8)
- U2 pad 9: unconnected-(U2-Pad9) -> Net-(U2-Pad9)
Routing:
- net VCC: track 0.00 -> 114.2 mm
- net Net-(U2-Pad28): track 0.00 -> 49.5 mm
- net Net-(U2-Pad27): track 0.00 -> 48.2 mm
- net Net-(D1-Pad2): track 0.00 -> 29.4 mm
- net Net-(D1-Pad1): track 0.00 -> 29.1 mm
- net +3V3: track 0.00 -> 27.7 mm
- net Net-(R2-Pad2): track 0.00 -> 26.4 mm
- net Net-(R5-Pad2): track 0.00 -> 18.2 mm
- net Net-(R4-Pad2): track 0.00 -> 14.1 mm
- net Net-(R3-Pad2): track 0.00 -> 11.8 mm
- net Net-(D2-Pad2): track 0.00 -> 10.4 mm
- net Net-(U2-Pad9): track 0.00 -> 10.2 mm
- net Net-(U2-Pad8): track 0.00 -> 10.2 mm
- net Net-(U2-Pad7): track 0.00 -> 10.2 mm
- net Net-(U2-Pad6): track 0.00 -> 10.2 mm
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- added copper zone on B.Cu, net GND
- added copper zone on F.Cu, net GND
